Commit message: Updated Arms, URDF, Added motion in Altair, etc.
- Updated URDF, now with legs, right arm, etc. (WIP)
- Tested Arm motion in Fusion360 & Altair Inspire.

File: Sim/RViz/humanoid_ws/src/humanoid_description/urdf/humanoid.urdf.xacro (robot description, xacro)
@@ -1,4 +1,5 @@
 <?xml version="1.0"?>
-<robot name= "humanoid" xmlns:xacro="http://www.ros.org/wiki/xacro">
+<robot name= "humanoid"
+    xmlns:xacro="http://www.ros.org/wiki/xacro">
     <!-- Constants -->
     <xacro:property name = "PI" value = "3.141593"/>
@@ -7,9 +8,15 @@
     <!-- Waist xacro -->
     <xacro:include filename="$(find humanoid_description)/urdf/waist.xacro"/>
+    <!-- Legs  xacro -->
+    <xacro:include filename="$(find humanoid_description)/urdf/humanoidrightleg.xacro"/>
+    <xacro:include filename="$(find humanoid_description)/urdf/humanoidleftleg.xacro"/>
+    <!-- Arm xacro -->
+    <xacro:include filename="$(find humanoid_description)/urdf/humanoidrightarm.xacro"/>
+    <!-- <xacro:include filename="$(find humanoid_description)/urdf/leg.xacro"/> -->
     <!-- World Link -->
     <link name="sim_world"/>
     <!-- base_link to world joint -->
     <joint name="base_link_sim_world_joint" type="fixed">
-        <origin xyz="0.0 0.0 0.0" rpy="${PI/2} 0.0 0.0"/>
+        <origin xyz="0.0 0.0 1.2" rpy="${PI/2} 0.0 0.0"/>
         <parent link="sim_world"/>
         <child link="torso"/>
@@ -19,3 +26,26 @@
         <origin xyz="-0.140001 -0.171194 0.05969" rpy="0 0 0"/>
     </xacro:waist_macro>
+    <!-- Right Leg -->
+    <xacro:rightleg_macro prefix = "RL" parent = "Right-femur-top_1">
+        <origin xyz="0.0 -0.074639 0.017302" rpy="0 0 0"/>
+    </xacro:rightleg_macro>
+    <!-- Left Leg -->
+    <xacro:leftleg_macro prefix = "LL" parent = "Left-femur-top_1">
+        <origin xyz="2e-06 -0.074639 -0.017302" rpy="0 0 0"/>
+    </xacro:leftleg_macro>
+    <!-- Right Arm-->
+    <xacro:arm_xacro prefix="RH" parent = "torso" sign = "1">
+        <origin xyz="-0.054627 0.160416 0.234212" rpy="0 0 ${-PI/2}"/>
+    </xacro:arm_xacro>
+    <!-- <xacro:arm_xacro prefix="LH" parent = "torso" sign = "1">
+        <origin xyz="-0.054536 0.160416 -0.114788" rpy="${PI} 0 0"/>
+    </xacro:arm_xacro> -->
+    <!-- Right Leg -->
+    <!-- <xacro:leg_macro prefix = "R" parent = "Right-femur-top_1" sign = "1">
+        <origin xyz="0.0 -0.074639 0.017302" rpy="0 0 0"/>
+    </xacro:leg_macro> -->
+    <!-- Left Leg -->
+    <!-- <xacro:leg_macro prefix = "L" parent = "Right-femur-top_1" sign = "-1">
+        <origin xyz="0 0 0" rpy="0 0 0"/>
+    </xacro:leg_macro> -->
 </robot>

File: Sim/RViz/humanoid_ws/src/humanoid_description/urdf/materials.xacro (robot description, xacro)
@@ -1,4 +1,4 @@
 <?xml version="1.0" ?>
-<robot name="torso" xmlns:xacro="http://www.ros.org/wiki/xacro" >
+<robot name="humanoid" xmlns:xacro="http://www.ros.org/wiki/xacro" >
 <material name="silver_default">
   <color rgba="0.700 0.700 0.700 1.000"/>
@@ -20,3 +20,35 @@
   <color rgba="1.0 0.6 0.0 1.0"/>
 </material>
+<!-- Leg Materials -->
+<material name="opaque22122113">
+  <color rgba="0.8666666666666667 0.8666666666666667 0.050980392156862744 1.0"/>
+</material>
+<material name="opaque191191191">
+  <color rgba="0.7490196078431373 0.7490196078431373 0.7490196078431373 1.0"/>
+</material>
+<material name="opaque252525">
+  <color rgba="0.09803921568627451 0.09803921568627451 0.09803921568627451 1.0"/>
+</material>
+<material name="opaque0125168">
+  <color rgba="0.0 0.49019607843137253 0.6588235294117647 1.0"/>
+</material>
+<material name="opaque2552550">
+  <color rgba="1.0 1.0 0.0 1.0"/>
+</material>
+<material name="opaque13110895">
+  <color rgba="0.5137254901960784 0.4235294117647059 0.37254901960784315 1.0"/>
+</material>
+<material name="powder_coat_green">
+  <color rgba="0.26666666666666666 0.5882352941176471 0.2823529411764706 0.0"/>
+</material>
+<!-- Hand Materials -->
+<material name="opaque808080">
+  <color rgba="0.3137254901960784 0.3137254901960784 0.3137254901960784 1.0"/>
+</material>
+<material name="opaque244244244">
+  <color rgba="0.9568627450980393 0.9568627450980393 0.9568627450980393 1.0"/>
+</material>
+<material name="opaque636363">
+  <color rgba="0.25098039215686274 0.25098039215686274 0.25098039215686274 1.0"/>
+</material>
 </robot>

File: Sim/RViz/humanoid_ws/src/humanoid_description/urdf/torso.xacro (robot description, xacro)
@@ -22,5 +22,5 @@
   </collision>
 </link>
-<link name="DumRArm_1">
+<!-- <link name="DumRArm_1">
   <inertial>
     <origin xyz="-2.461714795343184e-07 0.0007833561344568751 0.002499928901631726" rpy="0 0 0"/>
@@ -41,6 +41,6 @@
     </geometry>
   </collision>
-</link>
-<link name="DumLArm_1">
+</link> -->
+<!-- <link name="DumLArm_1">
   <inertial>
     <origin xyz="1.038923126056579e-06 0.0007833561272285461 -0.002500059100601068" rpy="0 0 0"/>
@@ -61,5 +61,5 @@
     </geometry>
   </collision>
-</link>
+</link> -->
 <link name="DumHead_1">
   <inertial>
@@ -82,16 +82,16 @@
   </collision>
 </link>
-<joint name="Revolute 5" type="continuous">
+<!-- <joint name="Revolute 5" type="continuous">
   <origin xyz="-0.054627 0.160416 0.234212" rpy="0 0 0"/>
   <parent link="torso"/>
   <child link="DumRArm_1"/>
   <axis xyz="-0.000261 0.0 1.0"/>
-</joint>
-<joint name="Revolute 6" type="continuous">
+</joint> -->
+<!-- <joint name="Revolute 6" type="continuous">
   <origin xyz="-0.054536 0.160416 -0.114788" rpy="0 0 0"/>
   <parent link="torso"/>
   <child link="DumLArm_1"/>
   <axis xyz="0.000261 -0.0 -1.0"/>
-</joint>
+</joint> -->
 <joint name="Rigid 7" type="fixed">
   <origin xyz="0.078519 0.116226 0.059747" rpy="0 0 0"/>

File: Sim/RViz/humanoid_ws/src/humanoid_description/urdf/waist.xacro (robot description, xacro)
@@ -82,5 +82,5 @@
     </collision>
   </link>
-  <link name="DumRightLeg_1">
+  <!-- <link name="DumRightLeg_1">
     <inertial>
       <origin xyz="-2.719365716774558e-07 -0.00043367314179110217 0.002461581106896815" rpy="0 0 0"/>
@@ -101,6 +101,6 @@
       </geometry>
     </collision>
-  </link>
-  <link name="DumLeftLeg_1">
+  </link> -->
+  <!-- <link name="DumLeftLeg_1">
     <inertial>
       <origin xyz="6.474975373111508e-07 -0.00043367314397685375 -0.0024621363755123714" rpy="0 0 0"/>
@@ -121,5 +121,5 @@
       </geometry>
     </collision>
-  </link>
+  </link> -->
   <link name="Buttocks_1">
     <inertial>
@@ -166,14 +166,14 @@
     <axis xyz="1.4e-05 -0.984808 -0.173648"/>
   </joint>
-  <joint name="Connection_to_R_leg" type="fixed">
+  <!-- <joint name="Connection_to_R_leg" type="fixed">
     <origin xyz="-7e-06 -0.074639 0.017302" rpy="0 0 0"/>
     <parent link="Right-femur-top_1"/>
     <child link="DumRightLeg_1"/>
-  </joint>
-  <joint name="Connection_to_L_leg" type="fixed">
+  </joint> -->
+  <!-- <joint name="Connection_to_L_leg" type="fixed">
     <origin xyz="2e-06 -0.074639 -0.017302" rpy="0 0 0"/>
     <parent link="Left-femur-top_1"/>
     <child link="DumLeftLeg_1"/>
-  </joint>
+  </joint> -->
   <joint name="torso_connection" type="fixed">
     <!-- <origin xyz="-0.140001 -0.171194 0.05969" rpy="0 0 0"/> -->
